Commit message: Main Package
Add some plugin to grasp objects, add python files to spawn model, pick and place specific items, count items and record files, and add a new moveit package for gripper

File: ur5_data_collect_fw/urdf/ur5_robot.urdf.xacro (robot description, xacro)
@@ -38,4 +38,7 @@
                 <box size="0.6 1.5 0.03"/>
             </geometry>
+            <material name="blue">
+                <color rgba="0 0 0.8 1"/>
+            </material>
         </visual>
         <collision>
@@ -48,5 +51,5 @@
         <mu1>0.2</mu1>
         <mu2>0.2</mu2>
-        <material>Gazebo/Yellow</material>
+        <material>Gazebo/Grass</material>
     </gazebo>
     <link name="box_sq">
@@ -60,6 +63,6 @@
                 <!-- <mesh filename="package://ur5_data_collect_fw/meshes/box_cc.stl" scale="0.001 0.001 0.001"/> -->
             </geometry>
-            <material name="silver">
-                <color rgba="0.700 0.700 0.700 1.000"/>
+            <material name="green">
+                <color rgba="0 0.8 0 1.000"/>
             </material>
         </visual>
@@ -71,5 +74,5 @@
     </link>
     <gazebo reference="box_sq">
-        <material>Gazebo/Silver</material>
+        <material>Gazebo/DarkMagentaTransparent</material>
         <mu1>0.2</mu1>
         <mu2>0.2</mu2>
@@ -124,4 +127,28 @@
         </collision>
     </link>
+    <gazebo reference="base_link">
+        <material>Gazebo/Yellow</material>
+    </gazebo>
+    <gazebo reference="shoulder_link">
+        <material>Gazebo/Yellow</material>
+    </gazebo>
+    <gazebo reference="upper_arm_link">
+        <material>Gazebo/Yellow</material>
+    </gazebo>
+    <gazebo reference="forearm_link">
+        <material>Gazebo/Yellow</material>
+    </gazebo>
+    <gazebo reference="wrist_1_link">
+        <material>Gazebo/Yellow</material>
+    </gazebo>
+    <gazebo reference="wrist_3_link">
+        <material>Gazebo/Yellow</material>
+    </gazebo>
+    <gazebo reference="wrist_2_link">
+        <material>Gazebo/Yellow</material>
+    </gazebo>
+    <gazebo reference="ee_link">
+        <material>Gazebo/Yellow</material>
+    </gazebo>
     <gazebo reference="ee_link2">
         <sensor name="ee_link2_contactsensor_sensor" type="contact">
@@ -136,3 +163,15 @@
         </sensor>
     </gazebo>
+    <link name="camera_frame"/>
+    <joint name="camera_frame_joint" type="fixed">
+        <parent link="world"/>
+        <child link="camera_frame"/>
+        <origin xyz="2.0 1.0 0.805" rpy="0.0 0.3 -2.6122"/>
+    </joint>
+    <link name="camera_depth_optical_frame"/>
+    <joint name="camera_depth_optical_frame_joint" type="fixed">
+        <parent link="camera_frame"/>
+        <child link="camera_depth_optical_frame"/>
+        <origin xyz="0.0 0.0 0.0" rpy="-1.5708 0 -1.5708"/>
+    </joint>
 </robot>
